File: test/test_out.brd (EAGLE design)
At the start: 100 x 100 mm, 36 parts

Commit message: tests: Update
Parts:
- renumbered E$11 to E$1_1, E$12 to E$1_2, E$13 to E$1_3, E$21 to E$2_1, E$22 to E$2_2, E$23 to E$2_3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
